Commit message: ur10 with a panda arm urdf

File: ur10e/ur10e.urdf (robot description, URDF)
Before this commit: robot ur10e, 8 links, 7 joints
Links:
- added link panda_grasptarget, mass 0.0
- added link panda_hand, mass .81; collision mesh filename=package://collision/hand.obj; visual mesh filename=package://visual/hand.obj
- added link panda_leftfinger, mass 0.1; collision mesh filename=package://collision/finger.obj; visual mesh filename=package://visual/finger.obj
- added link panda_rightfinger, mass 0.1; collision mesh filename=package://collision/finger.obj; visual mesh filename=package://visual/finger.obj
Joints:
- added joint panda_finger_joint1: type prismatic, parent panda_hand, child panda_leftfinger, origin xyz=0 0 0.0584 rpy=0 0 0, axis 0 1 0, limit lower=0.0 upper=0.04 effort=20 velocity=0.2
- added joint panda_finger_joint2: type prismatic, parent panda_hand, child panda_rightfinger, origin xyz=0 0 0.0584 rpy=0 0 0, axis 0 -1 0, limit lower=0.0 upper=0.04 effort=20 velocity=0.2, mimic joint=panda_finger_joint1
- added joint panda_grasptarget_hand: type fixed, parent panda_hand, child panda_grasptarget, origin xyz=0 0 0.105 rpy=0 0 0
- added joint panda_hand_joint: type fixed, parent tool0, child panda_hand, origin xyz=0 0 0 rpy=-1.57 0 0
